Commit message: 修改模型信息

File: catkin_ws/src/jetsonbot_description/urdf/jetsonbot_description.urdf (robot description, URDF)
Before this commit: robot jetsonbot_description, 5 links, 4 joints
Links:
- link base_link: mass 0.77436818932567 -> 0.77437
- link laser_link: mass 0.13782 -> 0.137819035246882
- link left_wheel_link: mass 0.048275 -> 0.0482752493266289
- link niujiaolun_link: mass 0.0091101 -> 0.00911013999938701
Joints:
- joint laser_joint: origin xyz=-0.043232 0.1765 0.00027141 rpy=0 0 0 -> xyz=-0.043232 -0.00027141 0.1765 rpy=0 0 0
- joint left_wheel_joint: axis 0 0 -1 -> 0 1 0; origin xyz=-0.043881 0.0215 -0.11073 rpy=0 0 0 -> xyz=-0.043881 0.11073 0.0215 rpy=0 0 0
- joint niujiaolun_joint: origin xyz=0.092152 -0.0059 0 rpy=0 0 0 -> xyz=0.092152 0 -0.0059 rpy=0 0 0
- joint right_wheel_joint: axis 0 0 -1 -> 0 1 0; origin xyz=-0.043881 0.0215 0.11073 rpy=0 0 0 -> xyz=-0.043881 -0.11073 0.0215 rpy=0 0 0
